File: latest/Presentation/boards/pedalboard-display.kicad_pcb (KiCad board)
At the start: 2 copper layers, 174 x 111 mm, 205 parts, among them J1 Conn_01x03_Pin, J2 Conn_01x03_Pin

Commit message: Deploying to main from @ pedalboard/pedalboard-display@f8f95626dab1886cdfae880860ee8407afd30411 🚀
Parts:
- removed DS1, DS2: OLED-128O064D, Display:OLED-128O064D
- added J3: OLED, Connector_JST:JST_PH_B4B-PH-SM4-TB_1x04-1MP_P2.00mm_Vertical, B.Cu at (127.0, 35.5)
- added U1: ~, Library:OLED_128x128, F.Cu at (63.2, 84.8)
- added U2: ~, Library:OLED_128x128, F.Cu at (146.3, 86.6)
