File: latest/Presentation/boards/pedalboard-display.kicad_pcb (KiCad board)
At the start: 2 copper layers, 174 x 111 mm, 206 parts, among them J1 LED-IN, J2 LED-OUT, J3 OLED

Commit message: Deploying to main from @ pedalboard/pedalboard-display@f11800b69cc1d232d4cb8142cff629dfbacd3cb2 🚀
Parts:
- added H1: MountingHole, MountingHole:MountingHole_2.5mm, F.Cu at (44.0, 28.0)
- added H2: MountingHole, MountingHole:MountingHole_2.5mm, F.Cu at (44.0, 133.0)
- added H3: MountingHole, MountingHole:MountingHole_2.5mm, F.Cu at (170.0, 28.0)
- added H4: MountingHole, MountingHole:MountingHole_2.5mm, F.Cu at (170.0, 133.0)
- added H5: MountingHole, MountingHole:MountingHole_2.5mm, F.Cu at (107.0, 103.0)
- turned C97 to -90 degrees

Commit message: Deploying to main from @ pedalboard/pedalboard-display@ed5daf3a73271a1219396e5281b2c6e43b89c100 🚀
Parts:
- moved C97 18.0 mm to (93.0, 53.0)
- moved C98 18.0 mm to (118.0, 53.0)
- moved D97 18.0 mm to (94.5, 53.0)
- moved D98 18.0 mm to (119.5, 53.0)
- moved J1 18.0 mm to (107.0, 53.0)
- moved R1 18.0 mm to (93.4, 51.5)
Routing:
- net /Led Ring GAIN/D_IN: track 49.8 -> 67.8 mm
- net /Led Ring E/D_OUT: track 89.9 -> 84.6 mm
- net +3.3V: track 108.8 -> 111.2 mm
- net /I2C_SDA: track 124.9 -> 127.3 mm
- net /I2C_SCL: track 109.9 -> 112.2 mm
- net /Led Ring B/D_IN: track 212.9 -> 211.6 mm
